Commit message: removed the steering links

File: ackermann_vehicle_description/urdf/model.urdf.xacro (robot description, xacro)
@@ -44,42 +44,16 @@
   <!-- - - - - - - - - - - - - - - - - - - - - - - - - - - - - - - - - - - -->
   <!-- FRONT -->
-  <!-- steering_link -->
-  <!-- left -->
-  <link name="left_steering_link">
-    <inertial>
-      <mass value="0.001"/>
-      <inertia ixx="0.001" ixy="0" ixz="0" iyy="0.001" iyz="0" izz="0.001"/>
-    </inertial>
-  </link>
-  <joint name="left_front_shock" type="fixed">
-    <parent link="chassis"/>
-    <child link="left_steering_link"/>
+  <!-- axel_carrier -->
+  <!-- left -->
+  <link name="left_front_axle_carrier">
+    <inertial>
+      <mass value="0.001"/>
+      <inertia ixx="0.001" ixy="0" ixz="0" iyy="0.001" iyz="0" izz="0.001"/>
+    </inertial>
+  </link>
+  <joint name="left_steering_joint" type="revolute">
+    <parent link="chassis"/>
+    <child link="left_front_axle_carrier"/>
     <origin xyz="0.1675 0.1525 -0.0235"/>
-    <axis xyz="0 0 -1"/>
-  </joint>
-  <!-- right -->
-  <link name="right_steering_link">
-    <inertial>
-      <mass value="0.001"/>
-      <inertia ixx="0.001" ixy="0" ixz="0" iyy="0.001" iyz="0" izz="0.001"/>
-    </inertial>
-  </link>
-  <joint name="right_front_shock" type="fixed">
-    <parent link="chassis"/>
-    <child link="right_steering_link"/>
-    <origin xyz="0.1675                    -0.1525                    -0.0235"/>
-    <axis xyz="0 0 -1"/>
-  </joint>
-  <!-- axel_carrier -->
-  <!-- left -->
-  <link name="left_front_axle_carrier">
-    <inertial>
-      <mass value="0.001"/>
-      <inertia ixx="0.001" ixy="0" ixz="0" iyy="0.001" iyz="0" izz="0.001"/>
-    </inertial>
-  </link>
-  <joint name="left_steering_joint" type="revolute">
-    <parent link="left_steering_link"/>
-    <child link="left_front_axle_carrier"/>
     <axis xyz="0 0 1"/>
     <limit effort="0.5649" lower="-0.785398163" upper="0.785398163" velocity="4.553"/>
@@ -102,6 +76,7 @@
   </link>
   <joint name="right_steering_joint" type="revolute">
-    <parent link="right_steering_link"/>
+    <parent link="chassis"/>
     <child link="right_front_axle_carrier"/>
+    <origin xyz="0.1675 -0.1525 -0.0235"/>
     <axis xyz="0 0 1"/>
     <limit effort="0.5649" lower="-0.785398163" upper="0.785398163" velocity="4.553"/>

Commit message: removed rear axle carrier

File: ackermann_vehicle_description/urdf/model.urdf.xacro (robot description, xacro)
@@ -172,31 +172,4 @@
   <!-- - - - - - - - - - - - - - - - - - - - - - - - - - - - - - - - - - - -->
   <!-- REAR -->
-  <!-- axle_carrier -->
-  <!-- left -->
-  <link name="left_rear_axle_carrier">
-    <inertial>
-      <mass value="0.001"/>
-      <inertia ixx="0.001" ixy="0" ixz="0" iyy="0.001" iyz="0" izz="0.001"/>
-    </inertial>
-  </link>
-  <joint name="left_rear_shock" type="fixed">
-    <parent link="chassis"/>
-    <child link="left_rear_axle_carrier"/>
-    <origin xyz="-0.1675                    0.1525                    -0.0235"/>
-    <axis xyz="0 0 -1"/>
-  </joint>
-  <!-- right -->
-  <link name="right_rear_axle_carrier">
-    <inertial>
-      <mass value="0.001"/>
-      <inertia ixx="0.001" ixy="0" ixz="0" iyy="0.001" iyz="0" izz="0.001"/>
-    </inertial>
-  </link>
-  <joint name="right_rear_shock" type="fixed">
-    <parent link="chassis"/>
-    <child link="right_rear_axle_carrier"/>
-    <origin xyz="-0.1675                    -0.1525                    -0.0235"/>
-    <axis xyz="0 0 -1"/>
-  </joint>
   <!-- wheels -->
   <!-- left -->
@@ -221,7 +194,7 @@
   </link>
   <joint name="left_rear_axle" type="continuous">
-    <parent link="left_rear_axle_carrier"/>
+    <parent link="chassis"/>
     <child link="left_rear_wheel"/>
-    <origin rpy="1.57079633 0 0"/>
+    <origin xyz="-0.1675 0.1525 -0.0235" rpy="1.57079633 0 0"/>
     <axis xyz="0 0 -1"/>
     <limit effort="5.12766" velocity="244.8696"/>
@@ -260,7 +233,7 @@
   </link>
   <joint name="right_rear_axle" type="continuous">
-    <parent link="right_rear_axle_carrier"/>
+    <parent link="chassis"/>
     <child link="right_rear_wheel"/>
-    <origin rpy="1.57079633 0 0"/>
+    <origin xyz="-0.1675 -0.1525 -0.0235" rpy="1.57079633 0 0"/>
     <axis xyz="0 0 -1"/>
     <limit effort="5.12766" velocity="244.8696"/>
