Commit message: launch at 0,0,0 and adjust chassis/base_link joint

File: ackermann_vehicle_description/urdf/barebones.urdf.xacro (robot description, xacro)
@@ -70,5 +70,5 @@
   <link name="chassis">
     <visual>
-      <origin xyz="0 0 ${-chassis_height/2}"/>
+      <origin xyz="0 0 0"/>
       <geometry>
         <box size="${chassis_length} ${chassis_width} ${chassis_height}"/>
@@ -77,5 +77,5 @@
     </visual>
     <collision>
-      <origin xyz="0 0 ${-chassis_height/2}"/>
+      <origin xyz="0 0 0"/>
       <geometry>
         <box size="${chassis_length} ${chassis_width} ${chassis_height}"/>
@@ -85,5 +85,5 @@
         width="${chassis_length}" depth="${chassis_width}"
         height="${chassis_height}" mass="${chassis_mass}">
-      <origin xyz="0 0 ${-chassis_height/2}"/>
+      <origin xyz="0 0 0"/>
     </xacro:solid_cuboid_inertial>
   </link>
@@ -91,4 +91,5 @@
     <parent link="base_link"/>
     <child link="chassis"/>
+    <origin xyz="0 0 ${chassis_height/2+tire_dia/2}"/>
   </joint>
   <gazebo reference="chassis">

Commit message: use more macro parameters, clean up

File: ackermann_vehicle_description/urdf/barebones.urdf.xacro (robot description, xacro)
@@ -17,9 +17,12 @@
   <xacro:property name="chassis_height" value="0.02"/>
   <xacro:property name="chassis_mass" value="2.788"/>
-  <!-- tire interial is a hollow cylinder, hence hub_dia -->
-  <xacro:property name="hub_dia" value="0.09652"/>
+  <!-- tire interia is a hollow cylinder, hence hub_dia -->
   <xacro:property name="tire_dia" value="0.14605"/>
+  <xacro:property name="hub_dia" value="${tire_dia/1.5}"/>
   <xacro:property name="tire_width" value="0.0889"/>
   <xacro:property name="wheel_mass" value="0.29"/>
+  <!-- wheel left/right and front/rear separation -->
+  <xacro:property name="wheel_lr_separation" value="${2*0.1525}"/>
+  <xacro:property name="wheel_fr_separation" value="${2*0.1675}"/>
   <!-- - - - - - - - - - - Inertia Macros - - - - - - - - - - -->
   <!-- Null -->
@@ -107,5 +110,5 @@
         <parent link="chassis"/>
         <child link="${lr_prefix}_front_axle_carrier"/>
-        <origin xyz="0.1675 ${lr_reflect*0.1525} 0"/>
+        <origin xyz="${wheel_fr_separation/2} ${lr_reflect*wheel_lr_separation/2} 0"/>
         <axis xyz="0 0 1"/>
         <limit effort="0.5649" lower="-0.785398163" upper="0.785398163" velocity="4.553"/>
@@ -189,5 +192,5 @@
         <parent link="chassis"/>
         <child link="${lr_prefix}_rear_wheel"/>
-        <origin xyz="-0.1675 ${lr_reflect*0.1525} 0" rpy="${pi/2} 0 0"/>
+        <origin xyz="${-wheel_fr_separation/2} ${lr_reflect*wheel_lr_separation/2} 0" rpy="${pi/2} 0 0"/>
         <axis xyz="0 0 -1"/>
         <limit effort="5.12766" velocity="244.8696"/>

Commit message: more macro parameters, clean up

File: ackermann_vehicle_description/urdf/barebones.urdf.xacro (robot description, xacro)
@@ -22,7 +22,10 @@
   <xacro:property name="tire_width" value="0.0889"/>
   <xacro:property name="wheel_mass" value="0.29"/>
-  <!-- wheel left/right and front/rear separation -->
-  <xacro:property name="wheel_lr_separation" value="${2*0.1525}"/>
-  <xacro:property name="wheel_fr_separation" value="${2*0.1675}"/>
+  <!-- tire left/right and front/rear separation -->
+  <xacro:property name="tire_lr_separation" value="${2*0.1525}"/>
+  <xacro:property name="tire_fr_separation" value="${2*0.1675}"/>
+  <!-- tire effort and veloicty -->
+  <xacro:property name="tire_effort" value="5.12766"/>
+  <xacro:property name="tire_velocity" value="244.8696"/>
   <!-- - - - - - - - - - - Inertia Macros - - - - - - - - - - -->
   <!-- Null -->
@@ -110,5 +113,5 @@
         <parent link="chassis"/>
         <child link="${lr_prefix}_front_axle_carrier"/>
-        <origin xyz="${wheel_fr_separation/2} ${lr_reflect*wheel_lr_separation/2} 0"/>
+        <origin xyz="${tire_fr_separation/2} ${lr_reflect*tire_lr_separation/2} 0"/>
         <axis xyz="0 0 1"/>
         <limit effort="0.5649" lower="-0.785398163" upper="0.785398163" velocity="4.553"/>
@@ -151,5 +154,5 @@
         <origin rpy="${pi/2} 0 0"/>
         <axis xyz="0 0 -1"/>
-        <limit effort="5.12766" velocity="244.8696"/>
+        <limit effort="${tire_effort}" velocity="${tire_velocity}"/>
     </joint>
     <transmission name="${lr_prefix}_front_axle_trans">
@@ -170,5 +173,5 @@
   <!-- - - - - - - - - - - - - - - - - - - - - - - - - - - - - - - - - - - -->
   <!-- REAR -->
-  <xacro:macro name="rear_wheel" params="lr_prefix lr_reflect">
+  <xacro:macro name="rear_tires" params="lr_prefix lr_reflect">
     <link name="${lr_prefix}_rear_wheel">
       <visual>
@@ -192,7 +195,7 @@
         <parent link="chassis"/>
         <child link="${lr_prefix}_rear_wheel"/>
-        <origin xyz="${-wheel_fr_separation/2} ${lr_reflect*wheel_lr_separation/2} 0" rpy="${pi/2} 0 0"/>
+        <origin xyz="${-tire_fr_separation/2} ${lr_reflect*tire_lr_separation/2} 0" rpy="${pi/2} 0 0"/>
         <axis xyz="0 0 -1"/>
-        <limit effort="5.12766" velocity="244.8696"/>
+        <limit effort="${tire_effort}" velocity="${tire_velocity}"/>
     </joint>
     <transmission name="${lr_prefix}_rear_axle_trans">
@@ -209,6 +212,6 @@
     </gazebo>
   </xacro:macro>
-  <xacro:rear_wheel lr_prefix="left" lr_reflect="1"/>
-  <xacro:rear_wheel lr_prefix="right" lr_reflect="-1"/>
+  <xacro:rear_tires lr_prefix="left" lr_reflect="1"/>
+  <xacro:rear_tires lr_prefix="right" lr_reflect="-1"/>
   <!-- gazebo plugins for control and odometry ground truth-->
   <gazebo>

Commit message: added macros for steering parameters

File: ackermann_vehicle_description/urdf/barebones.urdf.xacro (robot description, xacro)
@@ -12,5 +12,5 @@
   right -1
   -->
-  <!-- - - - - - - - - - - dimensions and mass - - - - - - - - - - -->
+  <!-- - - - - - - - - - dimensions, mass, and parameters - - - - - - - - - -->
   <xacro:property name="chassis_length" value="1.0"/>
   <xacro:property name="chassis_width" value="0.168"/>
@@ -25,7 +25,12 @@
   <xacro:property name="tire_lr_separation" value="${2*0.1525}"/>
   <xacro:property name="tire_fr_separation" value="${2*0.1675}"/>
-  <!-- tire effort and veloicty -->
+  <!-- tire parameters -->
   <xacro:property name="tire_effort" value="5.12766"/>
   <xacro:property name="tire_velocity" value="244.8696"/>
+  <!-- steeriing parameters -->
+  <xacro:property name="steeriing_effort" value="0.5649"/>
+  <xacro:property name="steeriing_lower" value="${-pi/4}"/>
+  <xacro:property name="steeriing_upper" value="${pi/4}"/>
+  <xacro:property name="steeriing_velocity" value="4.553"/>
   <!-- - - - - - - - - - - Inertia Macros - - - - - - - - - - -->
   <!-- Null -->
@@ -115,5 +120,5 @@
         <origin xyz="${tire_fr_separation/2} ${lr_reflect*tire_lr_separation/2} 0"/>
         <axis xyz="0 0 1"/>
-        <limit effort="0.5649" lower="-0.785398163" upper="0.785398163" velocity="4.553"/>
+        <limit effort="${steeriing_effort}" lower="${steeriing_lower}" upper="${steeriing_upper}" velocity="${steeriing_velocity}"/>
     </joint>
     <transmission name="${lr_prefix}_steering_trans">

Commit message: adjusted wheel separation, both lr and fr

File: ackermann_vehicle_description/urdf/barebones.urdf.xacro (robot description, xacro)
@@ -20,9 +20,9 @@
   <xacro:property name="tire_dia" value="0.14605"/>
   <xacro:property name="hub_dia" value="${tire_dia/1.5}"/>
-  <xacro:property name="tire_width" value="0.0889"/>
+  <xacro:property name="tire_width" value="${tire_dia/1.5}"/>
   <xacro:property name="wheel_mass" value="0.29"/>
   <!-- tire left/right and front/rear separation -->
-  <xacro:property name="tire_lr_separation" value="${2*0.1525}"/>
-  <xacro:property name="tire_fr_separation" value="${2*0.1675}"/>
+  <xacro:property name="tire_lr_separation" value="${chassis_width+tire_width}"/>
+  <xacro:property name="tire_fr_separation" value="${chassis_length}"/>
   <!-- tire parameters -->
   <xacro:property name="tire_effort" value="5.12766"/>

Commit message: mock truck parameters

File: ackermann_vehicle_description/urdf/barebones.urdf.xacro (robot description, xacro)
@@ -13,16 +13,17 @@
   -->
   <!-- - - - - - - - - - dimensions, mass, and parameters - - - - - - - - - -->
-  <xacro:property name="chassis_length" value="1.0"/>
-  <xacro:property name="chassis_width" value="0.168"/>
-  <xacro:property name="chassis_height" value="0.02"/>
+  <xacro:property name="chassis_length" value="3.38"/>
+  <xacro:property name="chassis_width" value="0.92"/>
+  <xacro:property name="chassis_height" value="1.4"/>
   <xacro:property name="chassis_mass" value="2.788"/>
   <!-- tire interia is a hollow cylinder, hence hub_dia -->
-  <xacro:property name="tire_dia" value="0.14605"/>
+  <xacro:property name="tire_dia" value="${0.575*2}"/>
   <xacro:property name="hub_dia" value="${tire_dia/1.5}"/>
-  <xacro:property name="tire_width" value="${tire_dia/1.5}"/>
+  <xacro:property name="tire_width" value="${tire_dia/3.0}"/>
   <xacro:property name="wheel_mass" value="0.29"/>
   <!-- tire left/right and front/rear separation -->
-  <xacro:property name="tire_lr_separation" value="${chassis_width+tire_width}"/>
-  <xacro:property name="tire_fr_separation" value="${chassis_length}"/>
+  <xacro:property name="tire_lr_separation" value="2.36"/>
+  <xacro:property name="tire_fr_separation" value="5.216"/>
+  <xacro:property name="tire_z_offset" value="${chassis_height/2+0.614}"/>
   <!-- tire parameters -->
   <xacro:property name="tire_effort" value="5.12766"/>
@@ -102,5 +103,5 @@
     <parent link="base_link"/>
     <child link="chassis"/>
-    <origin xyz="0 0 ${chassis_height/2+tire_dia/2}"/>
+    <origin xyz="0 0 ${tire_dia/2+tire_z_offset}"/>
   </joint>
   <gazebo reference="chassis">
@@ -118,5 +119,5 @@
         <parent link="chassis"/>
         <child link="${lr_prefix}_front_axle_carrier"/>
-        <origin xyz="${tire_fr_separation/2} ${lr_reflect*tire_lr_separation/2} 0"/>
+        <origin xyz="${tire_fr_separation/2} ${lr_reflect*tire_lr_separation/2} ${-tire_z_offset}"/>
         <axis xyz="0 0 1"/>
         <limit effort="${steeriing_effort}" lower="${steeriing_lower}" upper="${steeriing_upper}" velocity="${steeriing_velocity}"/>
@@ -200,5 +201,5 @@
         <parent link="chassis"/>
         <child link="${lr_prefix}_rear_wheel"/>
-        <origin xyz="${-tire_fr_separation/2} ${lr_reflect*tire_lr_separation/2} 0" rpy="${pi/2} 0 0"/>
+        <origin xyz="${-tire_fr_separation/2} ${lr_reflect*tire_lr_separation/2} ${-tire_z_offset}" rpy="${pi/2} 0 0"/>
         <axis xyz="0 0 -1"/>
         <limit effort="${tire_effort}" velocity="${tire_velocity}"/>

Commit message: wip: tyring to get the steering working on a large vehicle

File: ackermann_vehicle_description/urdf/barebones.urdf.xacro (robot description, xacro)
@@ -16,10 +16,10 @@
   <xacro:property name="chassis_width" value="0.92"/>
   <xacro:property name="chassis_height" value="1.4"/>
-  <xacro:property name="chassis_mass" value="2.788"/>
+  <xacro:property name="chassis_mass" value="1000"/>
   <!-- tire interia is a hollow cylinder, hence hub_dia -->
   <xacro:property name="tire_dia" value="${0.575*2}"/>
   <xacro:property name="hub_dia" value="${tire_dia/1.5}"/>
   <xacro:property name="tire_width" value="${tire_dia/3.0}"/>
-  <xacro:property name="wheel_mass" value="0.29"/>
+  <xacro:property name="wheel_mass" value="10"/>
   <!-- tire left/right and front/rear separation -->
   <xacro:property name="tire_lr_separation" value="2.36"/>
@@ -27,11 +27,16 @@
   <xacro:property name="tire_z_offset" value="${chassis_height/2+0.614}"/>
   <!-- tire parameters -->
-  <xacro:property name="tire_effort" value="5.12766"/>
-  <xacro:property name="tire_velocity" value="244.8696"/>
+  <xacro:property name="tire_effort" value="1000000"/>
+  <xacro:property name="tire_velocity" value="1000000"/>
+  <xacro:property name="tire_mu1" value="0.9"/>
+  <xacro:property name="tire_mu2" value="0.9"/>
+  <xacro:property name="tire_kp" value="${1e8}"/>
+  <!-- <xacro:property name="tire_kd" value="1.0"/> -->
+  <xacro:property name="tire_minDepth" value="0.005"/>
   <!-- steeriing parameters -->
-  <xacro:property name="steeriing_effort" value="0.5649"/>
+  <xacro:property name="steeriing_effort" value="10000000"/>
   <xacro:property name="steeriing_lower" value="${-pi/4}"/>
   <xacro:property name="steeriing_upper" value="${pi/4}"/>
-  <xacro:property name="steeriing_velocity" value="4.553"/>
+  <xacro:property name="steeriing_velocity" value="1000000"/>
   <!-- - - - - - - - - - - Inertia Macros - - - - - - - - - - -->
   <!-- Null -->
@@ -39,5 +44,5 @@
     <inertial>
       <mass value="0.001"/>
-      <inertia ixx="0.001" ixy="0" ixz="0" iyy="0.001" iyz="0" izz="0.001"/>
+      <inertia ixx="0.00001" ixy="0" ixz="0" iyy="0.00001" iyz="0" izz="0.00001"/>
     </inertial>
   </xacro:macro>
@@ -172,4 +177,9 @@
     </transmission>
     <gazebo reference="${lr_prefix}_front_wheel">
+        <mu1 value="${tire_mu1}"/>
+        <mu2 value="${tire_mu2}"/>
+        <kp value="${tire_kp}"/>
+        <!-- <kd value="${tire_kd}"/> -->
+        <minDepth value="${tire_minDepth}"/>
         <material>Gazebo/Black</material>
     </gazebo>
@@ -215,4 +225,9 @@
     </transmission>
     <gazebo reference="${lr_prefix}_rear_wheel">
+        <mu1 value="${tire_mu1}"/>
+        <mu2 value="${tire_mu2}"/>
+        <kp value="${tire_kp}"/>
+        <!-- <kd value="${tire_kd}"/> -->
+        <minDepth value="${tire_minDepth}"/>
         <material>Gazebo/Black</material>
     </gazebo>

Commit message: wip: tuning pid parameters

File: ackermann_vehicle_description/urdf/barebones.urdf.xacro (robot description, xacro)
@@ -16,5 +16,5 @@
   <xacro:property name="chassis_width" value="0.92"/>
   <xacro:property name="chassis_height" value="1.4"/>
-  <xacro:property name="chassis_mass" value="1000"/>
+  <xacro:property name="chassis_mass" value="500"/>
   <!-- tire interia is a hollow cylinder, hence hub_dia -->
   <xacro:property name="tire_dia" value="${0.575*2}"/>
@@ -27,6 +27,6 @@
   <xacro:property name="tire_z_offset" value="${chassis_height/2+0.614}"/>
   <!-- tire parameters -->
-  <xacro:property name="tire_effort" value="1000000"/>
-  <xacro:property name="tire_velocity" value="1000000"/>
+  <xacro:property name="tire_effort" value="100"/>
+  <xacro:property name="tire_velocity" value="10"/>
   <xacro:property name="tire_mu1" value="0.9"/>
   <xacro:property name="tire_mu2" value="0.9"/>
@@ -35,8 +35,8 @@
   <xacro:property name="tire_minDepth" value="0.005"/>
   <!-- steeriing parameters -->
-  <xacro:property name="steeriing_effort" value="10000000"/>
+  <xacro:property name="steeriing_effort" value="0"/>
   <xacro:property name="steeriing_lower" value="${-pi/4}"/>
   <xacro:property name="steeriing_upper" value="${pi/4}"/>
-  <xacro:property name="steeriing_velocity" value="1000000"/>
+  <xacro:property name="steeriing_velocity" value="0"/>
   <!-- - - - - - - - - - - Inertia Macros - - - - - - - - - - -->
   <!-- Null -->

Commit message: wip: works at slow speeds

File: ackermann_vehicle_description/urdf/barebones.urdf.xacro (robot description, xacro)
@@ -35,8 +35,8 @@
   <xacro:property name="tire_minDepth" value="0.005"/>
   <!-- steeriing parameters -->
-  <xacro:property name="steeriing_effort" value="0"/>
+  <xacro:property name="steeriing_effort" value="1000"/>
   <xacro:property name="steeriing_lower" value="${-pi/4}"/>
   <xacro:property name="steeriing_upper" value="${pi/4}"/>
-  <xacro:property name="steeriing_velocity" value="0"/>
+  <xacro:property name="steeriing_velocity" value="10"/>
   <!-- - - - - - - - - - - Inertia Macros - - - - - - - - - - -->
   <!-- Null -->

Commit message: wip: more weight

File: ackermann_vehicle_description/urdf/barebones.urdf.xacro (robot description, xacro)
@@ -16,10 +16,10 @@
   <xacro:property name="chassis_width" value="0.92"/>
   <xacro:property name="chassis_height" value="1.4"/>
-  <xacro:property name="chassis_mass" value="500"/>
+  <xacro:property name="chassis_mass" value="1000"/>
   <!-- tire interia is a hollow cylinder, hence hub_dia -->
   <xacro:property name="tire_dia" value="${0.575*2}"/>
   <xacro:property name="hub_dia" value="${tire_dia/1.5}"/>
   <xacro:property name="tire_width" value="${tire_dia/3.0}"/>
-  <xacro:property name="wheel_mass" value="10"/>
+  <xacro:property name="wheel_mass" value="50"/>
   <!-- tire left/right and front/rear separation -->
   <xacro:property name="tire_lr_separation" value="2.36"/>
@@ -35,5 +35,5 @@
   <xacro:property name="tire_minDepth" value="0.005"/>
   <!-- steeriing parameters -->
-  <xacro:property name="steeriing_effort" value="1000"/>
+  <xacro:property name="steeriing_effort" value="100000"/>
   <xacro:property name="steeriing_lower" value="${-pi/4}"/>
   <xacro:property name="steeriing_upper" value="${pi/4}"/>

Commit message: wip: still having problems tuning the pid and effort

File: ackermann_vehicle_description/urdf/barebones.urdf.xacro (robot description, xacro)
@@ -35,8 +35,8 @@
   <xacro:property name="tire_minDepth" value="0.005"/>
   <!-- steeriing parameters -->
-  <xacro:property name="steeriing_effort" value="100000"/>
+  <xacro:property name="steeriing_effort" value="1000000000000000"/>
   <xacro:property name="steeriing_lower" value="${-pi/4}"/>
   <xacro:property name="steeriing_upper" value="${pi/4}"/>
-  <xacro:property name="steeriing_velocity" value="10"/>
+  <xacro:property name="steeriing_velocity" value="0.1"/>
   <!-- - - - - - - - - - - Inertia Macros - - - - - - - - - - -->
   <!-- Null -->

Commit message: small wheels work just fine

File: ackermann_vehicle_description/urdf/barebones.urdf.xacro (robot description, xacro)
@@ -13,13 +13,21 @@
   -->
   <!-- - - - - - - - - - dimensions, mass, and parameters - - - - - - - - - -->
-  <xacro:property name="chassis_length" value="3.38"/>
+  <!-- <xacro:property name="chassis_length" value="3.38"/>
   <xacro:property name="chassis_width" value="0.92"/>
   <xacro:property name="chassis_height" value="1.4"/>
-  <xacro:property name="chassis_mass" value="1000"/>
+  <xacro:property name="chassis_mass" value="4"/> -->
+  <xacro:property name="chassis_length" value="0.258"/>
+  <xacro:property name="chassis_width" value="0.168"/>
+  <xacro:property name="chassis_height" value="0.02"/>
+  <xacro:property name="chassis_mass" value="2.788"/>
   <!-- tire interia is a hollow cylinder, hence hub_dia -->
-  <xacro:property name="tire_dia" value="${0.575*2}"/>
+  <!-- <xacro:property name="tire_dia" value="${0.575*2}"/>
   <xacro:property name="hub_dia" value="${tire_dia/1.5}"/>
   <xacro:property name="tire_width" value="${tire_dia/3.0}"/>
-  <xacro:property name="wheel_mass" value="50"/>
+  <xacro:property name="wheel_mass" value="1"/> -->
+  <xacro:property name="tire_dia" value="0.14605"/>
+  <xacro:property name="hub_dia" value="${tire_dia/1.5}"/>
+  <xacro:property name="tire_width" value="${tire_dia/3.0}"/>
+  <xacro:property name="wheel_mass" value="0.29"/>
   <!-- tire left/right and front/rear separation -->
   <xacro:property name="tire_lr_separation" value="2.36"/>
@@ -28,15 +36,15 @@
   <!-- tire parameters -->
   <xacro:property name="tire_effort" value="100"/>
-  <xacro:property name="tire_velocity" value="10"/>
-  <xacro:property name="tire_mu1" value="0.9"/>
-  <xacro:property name="tire_mu2" value="0.9"/>
-  <xacro:property name="tire_kp" value="${1e8}"/>
-  <!-- <xacro:property name="tire_kd" value="1.0"/> -->
-  <xacro:property name="tire_minDepth" value="0.005"/>
+  <xacro:property name="tire_velocity" value="100"/>
+  <xacro:property name="tire_mu1" value="1"/>
+  <xacro:property name="tire_mu2" value="1"/>
+  <xacro:property name="tire_kp" value="${1e9}"/>
+  <xacro:property name="tire_kd" value="${5e6}"/>
+  <!-- <xacro:property name="tire_minDepth" value="0.005"/> -->
   <!-- steeriing parameters -->
-  <xacro:property name="steeriing_effort" value="1000000000000000"/>
+  <xacro:property name="steeriing_effort" value="10000000"/>
   <xacro:property name="steeriing_lower" value="${-pi/4}"/>
   <xacro:property name="steeriing_upper" value="${pi/4}"/>
-  <xacro:property name="steeriing_velocity" value="0.1"/>
+  <xacro:property name="steeriing_velocity" value="10000000"/>
   <!-- - - - - - - - - - - Inertia Macros - - - - - - - - - - -->
   <!-- Null -->
@@ -180,6 +188,6 @@
         <mu2 value="${tire_mu2}"/>
         <kp value="${tire_kp}"/>
-        <!-- <kd value="${tire_kd}"/> -->
-        <minDepth value="${tire_minDepth}"/>
+        <kd value="${tire_kd}"/>
+        <!-- <minDepth value="${tire_minDepth}"/> -->
         <material>Gazebo/Black</material>
     </gazebo>
@@ -228,6 +236,6 @@
         <mu2 value="${tire_mu2}"/>
         <kp value="${tire_kp}"/>
-        <!-- <kd value="${tire_kd}"/> -->
-        <minDepth value="${tire_minDepth}"/>
+        <kd value="${tire_kd}"/>
+        <!-- <minDepth value="${tire_minDepth}"/> -->
         <material>Gazebo/Black</material>
     </gazebo>
