Commit message: working little wheels, large body

File: ackermann_vehicle_description/urdf/barebones.urdf.xacro (robot description, xacro)
@@ -13,21 +13,17 @@
   -->
   <!-- - - - - - - - - - dimensions, mass, and parameters - - - - - - - - - -->
-  <!-- <xacro:property name="chassis_length" value="3.38"/>
+  <xacro:property name="chassis_length" value="3.38"/>
   <xacro:property name="chassis_width" value="0.92"/>
   <xacro:property name="chassis_height" value="1.4"/>
-  <xacro:property name="chassis_mass" value="4"/> -->
-  <xacro:property name="chassis_length" value="0.258"/>
-  <xacro:property name="chassis_width" value="0.168"/>
-  <xacro:property name="chassis_height" value="0.02"/>
-  <xacro:property name="chassis_mass" value="2.788"/>
+  <xacro:property name="chassis_mass" value="4"/>
   <!-- tire interia is a hollow cylinder, hence hub_dia -->
   <!-- <xacro:property name="tire_dia" value="${0.575*2}"/>
   <xacro:property name="hub_dia" value="${tire_dia/1.5}"/>
-  <xacro:property name="tire_width" value="${tire_dia/3.0}"/>
-  <xacro:property name="wheel_mass" value="1"/> -->
+  <xacro:property name="tire_width" value="${tire_dia/3.0}"/> -->
+  <xacro:property name="wheel_mass" value="1"/>
   <xacro:property name="tire_dia" value="0.14605"/>
   <xacro:property name="hub_dia" value="${tire_dia/1.5}"/>
   <xacro:property name="tire_width" value="${tire_dia/3.0}"/>
-  <xacro:property name="wheel_mass" value="0.29"/>
+  <!-- <xacro:property name="wheel_mass" value="0.29"/> -->
   <!-- tire left/right and front/rear separation -->
   <xacro:property name="tire_lr_separation" value="2.36"/>
@@ -35,8 +31,8 @@
   <xacro:property name="tire_z_offset" value="${chassis_height/2+0.614}"/>
   <!-- tire parameters -->
-  <xacro:property name="tire_effort" value="100"/>
-  <xacro:property name="tire_velocity" value="100"/>
-  <xacro:property name="tire_mu1" value="1"/>
-  <xacro:property name="tire_mu2" value="1"/>
+  <xacro:property name="tire_effort" value="10000000"/>
+  <xacro:property name="tire_velocity" value="10000000"/>
+  <xacro:property name="tire_mu1" value="0.9"/>
+  <xacro:property name="tire_mu2" value="0.9"/>
   <xacro:property name="tire_kp" value="${1e9}"/>
   <xacro:property name="tire_kd" value="${5e6}"/>

Commit message: twice the little wheel diameter works just fine

File: ackermann_vehicle_description/urdf/barebones.urdf.xacro (robot description, xacro)
@@ -22,5 +22,5 @@
   <xacro:property name="tire_width" value="${tire_dia/3.0}"/> -->
   <xacro:property name="wheel_mass" value="1"/>
-  <xacro:property name="tire_dia" value="0.14605"/>
+  <xacro:property name="tire_dia" value="${2*0.14605}"/>
   <xacro:property name="hub_dia" value="${tire_dia/1.5}"/>
   <xacro:property name="tire_width" value="${tire_dia/3.0}"/>

Commit message: 4x larger tires, problems are showing, I think the PID needs to be tuned

File: ackermann_vehicle_description/urdf/barebones.urdf.xacro (robot description, xacro)
@@ -22,5 +22,5 @@
   <xacro:property name="tire_width" value="${tire_dia/3.0}"/> -->
   <xacro:property name="wheel_mass" value="1"/>
-  <xacro:property name="tire_dia" value="${2*0.14605}"/>
+  <xacro:property name="tire_dia" value="${4*0.14605}"/>
   <xacro:property name="hub_dia" value="${tire_dia/1.5}"/>
   <xacro:property name="tire_width" value="${tire_dia/3.0}"/>

Commit message: large wheels and tuned PID

File: ackermann_vehicle_description/urdf/barebones.urdf.xacro (robot description, xacro)
@@ -22,5 +22,5 @@
   <xacro:property name="tire_width" value="${tire_dia/3.0}"/> -->
   <xacro:property name="wheel_mass" value="1"/>
-  <xacro:property name="tire_dia" value="${4*0.14605}"/>
+  <xacro:property name="tire_dia" value="${8*0.14605}"/>
   <xacro:property name="hub_dia" value="${tire_dia/1.5}"/>
   <xacro:property name="tire_width" value="${tire_dia/3.0}"/>

Commit message: truck parameters used

File: ackermann_vehicle_description/urdf/barebones.urdf.xacro (robot description, xacro)
@@ -18,12 +18,8 @@
   <xacro:property name="chassis_mass" value="4"/>
   <!-- tire interia is a hollow cylinder, hence hub_dia -->
-  <!-- <xacro:property name="tire_dia" value="${0.575*2}"/>
-  <xacro:property name="hub_dia" value="${tire_dia/1.5}"/>
-  <xacro:property name="tire_width" value="${tire_dia/3.0}"/> -->
-  <xacro:property name="wheel_mass" value="1"/>
-  <xacro:property name="tire_dia" value="${8*0.14605}"/>
+  <xacro:property name="tire_dia" value="${0.575*2}"/>
   <xacro:property name="hub_dia" value="${tire_dia/1.5}"/>
   <xacro:property name="tire_width" value="${tire_dia/3.0}"/>
-  <!-- <xacro:property name="wheel_mass" value="0.29"/> -->
+  <xacro:property name="wheel_mass" value="1"/>
   <!-- tire left/right and front/rear separation -->
   <xacro:property name="tire_lr_separation" value="2.36"/>
